Commit message: Parametize serial port

File: config/ar3.ros2_control.xacro (robot description, xacro)
@@ -1,13 +1,11 @@
 <?xml version="1.0"?>
 <robot xmlns:xacro="http://www.ros.org/wiki/xacro">
-    <xacro:macro name="ar3_ros2_control" params="name initial_positions_file">
+    <xacro:macro name="ar3_ros2_control" params="name initial_positions_file serial_port baud_rate">
         <xacro:property name="initial_positions" value="${load_yaml(initial_positions_file)['initial_positions']}"/>
         <ros2_control name="${name}" type="system">
             <hardware>
-                <!-- By default, set up controllers for simulation. This won't work on real hardware -->
-                <!-- <plugin>mock_components/GenericSystem</plugin> -->
                 <plugin>ar3_hardware_interface/AR3HardwareInterface</plugin>
-                <param name="serial_port">/dev/ttyCobot0</param>
-                <param name="baud_rate">115200</param>
+                <param name="serial_port">${serial_port}</param>
+                <param name="baud_rate">${baud_rate}</param>
             </hardware>
             <joint name="joint_0">

File: config/ar3.urdf.xacro (robot description, xacro)
@@ -2,8 +2,10 @@
 <robot xmlns:xacro="http://www.ros.org/wiki/xacro" name="ar3">
     <xacro:arg name="initial_positions_file" default="initial_positions.yaml" />
+    <xacro:arg name="serial_port" default="/dev/ttyCobot0" />
+    <xacro:arg name="baud_rate" default="115200" />
     <!-- Import ar3 urdf file -->
     <xacro:include filename="$(find ar3_description)/urdf/ar3.urdf.xacro" />
     <!-- Import control_xacro -->
     <xacro:include filename="ar3.ros2_control.xacro" />
-    <xacro:ar3_ros2_control name="ar3_system" initial_positions_file="$(arg initial_positions_file)"/>
+    <xacro:ar3_ros2_control name="ar3_system" initial_positions_file="$(arg initial_positions_file)" serial_port="$(arg serial_port)" baud_rate="$(arg baud_rate)"/>
 </robot>
