Commit message: Add bias

File: single-cobot-moveit-config/config/cobot0.ros2_control.xacro (robot description, xacro)
@@ -69,4 +69,40 @@
                 </state_interface>
             </joint>
+            <joint name="cobot0_joint_0_bias">
+                <command_interface name="position"/>
+                <state_interface name="position">
+                  <param name="initial_value">0</param>
+                </state_interface>
+            </joint>
+            <joint name="cobot0_joint_1_bias">
+                <command_interface name="position"/>
+                <state_interface name="position">
+                  <param name="initial_value">0</param>
+                </state_interface>
+            </joint>
+            <joint name="cobot0_joint_2_bias">
+                <command_interface name="position"/>
+                <state_interface name="position">
+                  <param name="initial_value">0</param>
+                </state_interface>
+            </joint>
+            <joint name="cobot0_joint_3_bias">
+                <command_interface name="position"/>
+                <state_interface name="position">
+                  <param name="initial_value">0</param>
+                </state_interface>
+            </joint>
+            <joint name="cobot0_joint_4_bias">
+                <command_interface name="position"/>
+                <state_interface name="position">
+                  <param name="initial_value">0</param>
+                </state_interface>
+            </joint>
+            <joint name="cobot0_joint_5_bias">
+                <command_interface name="position"/>
+                <state_interface name="position">
+                  <param name="initial_value">0</param>
+                </state_interface>
+            </joint>
         </ros2_control>
     </xacro:macro>
